Commit message: change the finger tip to be fixed

File: data/kinova_kg3/kinova_kg3.urdf (robot description, URDF)
Before this commit: robot kinova_kg3, 7 links, 6 joints
Links:
- removed link jaco_link_finger_tip_1
- removed link jaco_link_finger_tip_2
- removed link jaco_link_finger_tip_3
- link jaco_link_finger_1: mass 0.0008862 -> 0.0021306
- link jaco_link_finger_2: mass 0.0008862 -> 0.0021306
- link jaco_link_finger_3: mass 0.0008862 -> 0.0021306
Joints:
- removed joint jaco_joint_finger_tip_1
- removed joint jaco_joint_finger_tip_2
- removed joint jaco_joint_finger_tip_3

File: data/kinova_kg3/kinova_kg3_finger.xacro (robot description, xacro)
@@ -16,12 +16,12 @@
 			<inertial>
 			  <origin
-				  xyz="${0.208232/MESHLAB_SCALE} ${-0.062151/MESHLAB_SCALE} ${0.000043/MESHLAB_SCALE}"
+				  xyz="${0.426520/MESHLAB_SCALE} ${-0.061351/MESHLAB_SCALE} ${0.000022/MESHLAB_SCALE}"
 				rpy="0 0 0" />
-			  <mass value="${0.008862/MESHLAB_SCALE}" />
+			  <mass value="${0.021306/MESHLAB_SCALE}" />
 		      <inertia
-				  ixx="${0.000104/MESHLAB_SCALE/MESHLAB_SCALE}"
-				  iyy="${0.000239/MESHLAB_SCALE/MESHLAB_SCALE}"
-				  izz="${0.000218/MESHLAB_SCALE/MESHLAB_SCALE}"
-				  ixy="${-0.000013/MESHLAB_SCALE/MESHLAB_SCALE}"
+				  ixx="${0.000172/MESHLAB_SCALE/MESHLAB_SCALE}"
+				  iyy="${0.001210/MESHLAB_SCALE/MESHLAB_SCALE}"
+				  izz="${0.001179/MESHLAB_SCALE/MESHLAB_SCALE}"
+				  ixy="${0.000012/MESHLAB_SCALE/MESHLAB_SCALE}"
 				  ixz="${0.0/MESHLAB_SCALE/MESHLAB_SCALE}"
 				  iyz="${0.0/MESHLAB_SCALE/MESHLAB_SCALE}"
@@ -44,40 +44,4 @@
 			</collision>
 	    </link>
-		<link name="jaco_link_finger_tip_${index}">
-			<inertial>
-			  <origin
-				xyz="${0.140432/MESHLAB_SCALE} ${-0.060580/MESHLAB_SCALE} ${0.000007/MESHLAB_SCALE}"
-				rpy="0 0 0" />
-			  <mass value="0.0124078189139213" />
-		      <inertia
-				  ixx="${0.000068/MESHLAB_SCALE/MESHLAB_SCALE}"
-				  iyy="${0.000247/MESHLAB_SCALE/MESHLAB_SCALE}"
-				  izz="${0.000236/MESHLAB_SCALE/MESHLAB_SCALE}"
-				  ixy="${0.000028/MESHLAB_SCALE/MESHLAB_SCALE}"
-				  ixz="${0.0/MESHLAB_SCALE/MESHLAB_SCALE}"
-				  iyz="${0.0/MESHLAB_SCALE/MESHLAB_SCALE}"
-			  />
-	        </inertial>
-			<visual>
-			  <origin xyz="0 0 0" rpy="0 0 0" />
-			  <geometry>
-				  <mesh filename="${PKG}meshes/jaco_link_finger_tip_2.STL" />
-			  </geometry>
-			  <material name="kinova_color"/>
-			</visual>
-			<collision>
-			  <origin xyz="0 0 0" rpy="0 0 0" />
-			  <geometry>
-				  <mesh filename="${PKG}meshes/jaco_link_finger_tip_2.STL" />
-			  </geometry>
-			</collision>
-		</link>
-		<joint name="jaco_joint_finger_tip_${index}" type="revolute">
-		    <origin xyz="0.0441021541423999 0 0" rpy="-1.11022302462516E-16 1.38777878078145E-17 -8.67361737988404E-18" />
-			<parent link="jaco_link_finger_${index}" />
-			<child link="jaco_link_finger_tip_${index}" />
-			<limit lower="0" upper="${50*M_PI/180}" effort="30" velocity="5"/>
-			<axis xyz="0 0 1" />
-		</joint>
 	</xacro:macro>
 </robot>

Commit message: simplify the stl collision files

File: data/kinova_kg3/kinova_kg3.urdf (robot description, URDF)
Before this commit: robot kinova_kg3, 4 links, 3 joints
Links:
- link jaco_link_finger_1: geometry collision mesh filename=meshes/jaco_link_finger_2_collision.STL; visual mesh filename=meshes/jaco_link_finger_2.STL
- link jaco_link_finger_2: geometry collision mesh filename=meshes/jaco_link_finger_2_collision.STL; visual mesh filename=meshes/jaco_link_finger_2.STL
- link jaco_link_finger_3: geometry collision mesh filename=meshes/jaco_link_finger_2_collision.STL; visual mesh filename=meshes/jaco_link_finger_2.STL
- link jaco_link_hand: geometry collision mesh filename=meshes/jaco_link_hand_collision.STL; visual mesh filename=meshes/jaco_link_hand.STL

File: data/kinova_kg3/kinova_kg3.xacro (robot description, xacro)
@@ -75,5 +75,5 @@
 		  <origin xyz="0 0 0" rpy="0 0 0" />
 		  <geometry>
-			  <mesh filename="${PKG}meshes/jaco_link_hand.STL" />
+			  <mesh filename="${PKG}meshes/jaco_link_hand_collision.STL" />
 		  </geometry>
 		</collision>

File: data/kinova_kg3/kinova_kg3_finger.xacro (robot description, xacro)
@@ -40,5 +40,5 @@
 			  <origin xyz="0 0 0" rpy="0 0 0" />
 			  <geometry>
-				  <mesh filename="${PKG}meshes/jaco_link_finger_2.STL" />
+				  <mesh filename="${PKG}meshes/jaco_link_finger_2_collision.STL" />
 			  </geometry>
 			</collision>
